Commit message: 6_6

File: resources/franka_convert.urdf (robot description, URDF)
Before this commit: robot panda, 12 links, 11 joints
Links:
- link panda_hand: geometry collision mesh filename=file:///home/franka/home/rfmove_workspace/rfmove/resources/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; visual mesh filename=file:///home/franka/home/rfmove_workspace/rfmove/resources/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
- link panda_leftfinger: geometry collision mesh filename=file:///home/franka/home/rfmove_workspace/rfmove/resources/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; visual mesh filename=file:///home/franka/home/rfmove_workspace/rfmove/resources/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
- link panda_link0: geometry collision mesh filename=file:///home/franka/home/rfmove_workspace/rfmove/resources/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; visual mesh filename=file:///home/franka/home/rfmove_workspace/rfmove/resources/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
- link panda_link1: geometry collision mesh filename=file:///home/franka/home/rfmove_workspace/rfmove/resources/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; visual mesh filename=file:///home/franka/home/rfmove_workspace/rfmove/resources/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
- link panda_link2: geometry collision mesh filename=file:///home/franka/home/rfmove_workspace/rfmove/resources/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; visual mesh filename=file:///home/franka/home/rfmove_workspace/rfmove/resources/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
- link panda_link3: geometry collision mesh filename=file:///home/franka/home/rfmove_workspace/rfmove/resources/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; visual mesh filename=file:///home/franka/home/rfmove_workspace/rfmove/resources/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
- link panda_link4: geometry collision mesh filename=file:///home/franka/home/rfmove_workspace/rfmove/resources/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; visual mesh filename=file:///home/franka/home/rfmove_workspace/rfmove/resources/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
- link panda_link5: geometry collision mesh filename=file:///home/franka/home/rfmove_workspace/rfmove/resources/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; visual mesh filename=file:///home/franka/home/rfmove_workspace/rfmove/resources/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
- link panda_link6: geometry collision mesh filename=file:///home/franka/home/rfmove_workspace/rfmove/resources/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; visual mesh filename=file:///home/franka/home/rfmove_workspace/rfmove/resources/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
- link panda_link7: geometry collision mesh filename=file:///home/franka/home/rfmove_workspace/rfmove/resources/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; visual mesh filename=file:///home/franka/home/rfmove_workspace/rfmove/resources/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
- link panda_rightfinger: geometry collision mesh filename=file:///home/franka/home/rfmove_workspace/rfmove/resources/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; visual mesh filename=file:///home/franka/home/rfmove_workspace/rfmove/resources/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

Commit message: 6_13

File: resources/franka_convert.urdf (robot description, URDF)
Before this commit: robot panda, 12 links, 11 joints
Links:
- link panda_hand: geometry collision mesh filename=file:///home/lees/linux_bak/rfmove/resources/franka_descrip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; visual mesh filename=file:///home/lees/linux_bak/rfmove/resources/franka_descrip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
- link panda_leftfinger: geometry collision mesh filename=file:///home/lees/linux_bak/rfmove/resources/franka_descrip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; visual mesh filename=file:///home/lees/linux_bak/rfmove/resources/franka_descrip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
- link panda_link0: geometry collision mesh filename=file:///home/lees/linux_bak/rfmove/resources/franka_descrip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; visual mesh filename=file:///home/lees/linux_bak/rfmove/resources/franka_descrip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
- link panda_link1: geometry collision mesh filename=file:///home/lees/linux_bak/rfmove/resources/franka_descrip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; visual mesh filename=file:///home/lees/linux_bak/rfmove/resources/franka_descrip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
- link panda_link2: geometry collision mesh filename=file:///home/lees/linux_bak/rfmove/resources/franka_descrip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; visual mesh filename=file:///home/lees/linux_bak/rfmove/resources/franka_descrip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
- link panda_link3: geometry collision mesh filename=file:///home/lees/linux_bak/rfmove/resources/franka_descrip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; visual mesh filename=file:///home/lees/linux_bak/rfmove/resources/franka_descrip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
- link panda_link4: geometry collision mesh filename=file:///home/lees/linux_bak/rfmove/resources/franka_descrip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; visual mesh filename=file:///home/lees/linux_bak/rfmove/resources/franka_descrip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
- link panda_link5: geometry collision mesh filename=file:///home/lees/linux_bak/rfmove/resources/franka_descrip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; visual mesh filename=file:///home/lees/linux_bak/rfmove/resources/franka_descrip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
- link panda_link6: geometry collision mesh filename=file:///home/lees/linux_bak/rfmove/resources/franka_descrip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; visual mesh filename=file:///home/lees/linux_bak/rfmove/resources/franka_descrip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
- link panda_link7: geometry collision mesh filename=file:///home/lees/linux_bak/rfmove/resources/franka_descrip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; visual mesh filename=file:///home/lees/linux_bak/rfmove/resources/franka_descrip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
- link panda_rightfinger: geometry collision mesh filename=file:///home/lees/linux_bak/rfmove/resources/franka_descrip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; visual mesh filename=file:///home/lees/linux_bak/rfmove/resources/franka_descrip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

Commit message: rfmove_6_20

File: resources/franka_convert.urdf (robot description, URDF)
Before this commit: robot panda, 12 links, 11 joints
Links:
- link panda_hand: geometry collision mesh filename=file:///home/ziye01/rfmove/resources/franka_description/mes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; visual mesh filename=file:///home/ziye01/rfmove/resources/franka_description/mes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
- link panda_leftfinger: geometry collision mesh filename=file:///home/ziye01/rfmove/resources/franka_description/mes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; visual mesh filename=file:///home/ziye01/rfmove/resources/franka_description/mes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
- link panda_link0: geometry collision mesh filename=file:///home/ziye01/rfmove/resources/franka_description/mes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; visual mesh filename=file:///home/ziye01/rfmove/resources/franka_description/mes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
- link panda_link1: geometry collision mesh filename=file:///home/ziye01/rfmove/resources/franka_description/mes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; visual mesh filename=file:///home/ziye01/rfmove/resources/franka_description/mes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
- link panda_link2: geometry collision mesh filename=file:///home/ziye01/rfmove/resources/franka_description/mes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; visual mesh filename=file:///home/ziye01/rfmove/resources/franka_description/mes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
- link panda_link3: geometry collision mesh filename=file:///home/ziye01/rfmove/resources/franka_description/mes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; visual mesh filename=file:///home/ziye01/rfmove/resources/franka_description/mes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
- link panda_link4: geometry collision mesh filename=file:///home/ziye01/rfmove/resources/franka_description/mes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; visual mesh filename=file:///home/ziye01/rfmove/resources/franka_description/mes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
- link panda_link5: geometry collision mesh filename=file:///home/ziye01/rfmove/resources/franka_description/mes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; visual mesh filename=file:///home/ziye01/rfmove/resources/franka_description/mes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
- link panda_link6: geometry collision mesh filename=file:///home/ziye01/rfmove/resources/franka_description/mes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; visual mesh filename=file:///home/ziye01/rfmove/resources/franka_description/mes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
- link panda_link7: geometry collision mesh filename=file:///home/ziye01/rfmove/resources/franka_description/mes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; visual mesh filename=file:///home/ziye01/rfmove/resources/franka_description/mes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
- link panda_rightfinger: geometry collision mesh filename=file:///home/ziye01/rfmove/resources/franka_description/mes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; visual mesh filename=file:///home/ziye01/rfmove/resources/franka_description/mes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
