Commit message: rfmove_7_3

File: resources/franka/urdf/franka_convert.urdf (robot description, URDF)
Before this commit: robot panda, 12 links, 11 joints
Links:
- link panda_hand: geometry collision mesh filename=file:///home/ziye01/rfmove/resources/franka/franka_descript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; visual mesh filename=file:///home/ziye01/rfmove/resources/franka/franka_descript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
- link panda_leftfinger: geometry collision mesh filename=file:///home/ziye01/rfmove/resources/franka/franka_descript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; visual mesh filename=file:///home/ziye01/rfmove/resources/franka/franka_descript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
- link panda_link0: geometry collision mesh filename=file:///home/ziye01/rfmove/resources/franka/franka_descript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; visual mesh filename=file:///home/ziye01/rfmove/resources/franka/franka_descript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
- link panda_link1: geometry collision mesh filename=file:///home/ziye01/rfmove/resources/franka/franka_descript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; visual mesh filename=file:///home/ziye01/rfmove/resources/franka/franka_descript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
- link panda_link2: geometry collision mesh filename=file:///home/ziye01/rfmove/resources/franka/franka_descript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; visual mesh filename=file:///home/ziye01/rfmove/resources/franka/franka_descript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
- link panda_link3: geometry collision mesh filename=file:///home/ziye01/rfmove/resources/franka/franka_descript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; visual mesh filename=file:///home/ziye01/rfmove/resources/franka/franka_descript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
- link panda_link4: geometry collision mesh filename=file:///home/ziye01/rfmove/resources/franka/franka_descript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; visual mesh filename=file:///home/ziye01/rfmove/resources/franka/franka_descript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
- link panda_link5: geometry collision mesh filename=file:///home/ziye01/rfmove/resources/franka/franka_descript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; visual mesh filename=file:///home/ziye01/rfmove/resources/franka/franka_descript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
- link panda_link6: geometry collision mesh filename=file:///home/ziye01/rfmove/resources/franka/franka_descript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; visual mesh filename=file:///home/ziye01/rfmove/resources/franka/franka_descript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
- link panda_link7: geometry collision mesh filename=file:///home/ziye01/rfmove/resources/franka/franka_descript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; visual mesh filename=file:///home/ziye01/rfmove/resources/franka/franka_descript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
- link panda_rightfinger: geometry collision mesh filename=file:///home/ziye01/rfmove/resources/franka/franka_descript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; visual mesh filename=file:///home/ziye01/rfmove/resources/franka/franka_descript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

File: resources/tobor/tobor_description/tobor.urdf (robot description, URDF)
Before this commit: robot r300, 71 links, 70 joints
Links:
- link PTZ_axis_link: geometry collision mesh filename=file:///home/ziye01/rfmove/resources/tobor/tobor_descriptio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; visual mesh filename=file:///home/ziye01/rfmove/resources/tobor/tobor_descriptio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
- link PTZ_base_link: geometry collision mesh filename=file:///home/ziye01/rfmove/resources/tobor/tobor_descriptio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; visual mesh filename=file:///home/ziye01/rfmove/resources/tobor/tobor_descriptio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
- link PTZ_camera_link: geometry collision box size=0.02505 0.09 0.025; visual mesh filename=file:///home/ziye01/rfmove/resources/tobor/tobor_descriptio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
- link PTZ_head_link: geometry collision mesh filename=file:///home/ziye01/rfmove/resources/tobor/tobor_descriptio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; visual mesh filename=file:///home/ziye01/rfmove/resources/tobor/tobor_descriptio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
- link PTZ_link: geometry collision mesh filename=file:///home/ziye01/rfmove/resources/tobor/tobor_descriptio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; visual mesh filename=file:///home/ziye01/rfmove/resources/tobor/tobor_descriptio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
- link base_link: mass 0.0001 -> None; geometry collision mesh filename=file:///home/ziye01/rfmove/resources/tobor/tobor_descriptio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; visual mesh filename=file:///home/ziye01/rfmove/resources/tobor/tobor_descriptio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
- link battery_cover_link: geometry collision mesh filename=file:///home/ziye01/rfmove/resources/tobor/tobor_descriptio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; visual mesh filename=file:///home/ziye01/rfmove/resources/tobor/tobor_descriptio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
- link cylinder_link: geometry collision mesh filename=file:///home/ziye01/rfmove/resources/tobor/tobor_descriptio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; visual mesh filename=file:///home/ziye01/rfmove/resources/tobor/tobor_descriptio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
- link driven_gear_link: geometry collision mesh filename=file:///home/ziye01/rfmove/resources/tobor/tobor_descriptio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; visual mesh filename=file:///home/ziye01/rfmove/resources/tobor/tobor_descriptio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
- link driving_gear_link: geometry collision mesh filename=file:///home/ziye01/rfmove/resources/tobor/tobor_descriptio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; visual mesh filename=file:///home/ziye01/rfmove/resources/tobor/tobor_descriptio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
- link electric_cylinder_base_link: geometry collision mesh filename=file:///home/ziye01/rfmove/resources/tobor/tobor_descriptio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; visual mesh filename=file:///home/ziye01/rfmove/resources/tobor/tobor_descriptio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
- link fixed_PTZ_link: geometry collision mesh filename=file:///home/ziye01/rfmove/resources/tobor/tobor_descriptio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; visual mesh filename=file:///home/ziye01/rfmove/resources/tobor/tobor_descriptio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
- link fixed_frame_link: geometry collision mesh filename=file:///home/ziye01/rfmove/resources/tobor/tobor_descriptio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; visual mesh filename=file:///home/ziye01/rfmove/resources/tobor/tobor_descriptio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
- link front_low_body_link: geometry collision mesh filename=file:///home/ziye01/rfmove/resources/tobor/tobor_descriptio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; visual mesh filename=file:///home/ziye01/rfmove/resources/tobor/tobor_descriptio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
- link front_upper_body_link: geometry collision mesh filename=file:///home/ziye01/rfmove/resources/tobor/tobor_descriptio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; visual mesh filename=file:///home/ziye01/rfmove/resources/tobor/tobor_descriptio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
- link left_arm_base: geometry collision mesh filename=file:///home/ziye01/rfmove/resources/tobor/tobor_descriptio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 scale=0.001 0.001 0.001; visual mesh filename=file:///home/ziye01/rfmove/resources/tobor/tobor_descriptio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 scale=0.001 0.001 0.001
- link left_arm_link1: geometry collision mesh filename=file:///home/ziye01/rfmove/resources/tobor/tobor_descriptio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 scale=0.001 0.001 0.001; visual mesh filename=file:///home/ziye01/rfmove/resources/tobor/tobor_descriptio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 scale=0.001 0.001 0.001
- link left_arm_link2: geometry collision mesh filename=file:///home/ziye01/rfmove/resources/tobor/tobor_descriptio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 scale=0.001 0.001 0.001; visual mesh filename=file:///home/ziye01/rfmove/resources/tobor/tobor_descriptio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 scale=0.001 0.001 0.001
- link left_arm_link3: geometry collision mesh filename=file:///home/ziye01/rfmove/resources/tobor/tobor_descriptio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 scale=0.001 0.001 0.001; visual mesh filename=file:///home/ziye01/rfmove/resources/tobor/tobor_descriptio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 scale=0.001 0.001 0.001
- link left_arm_link4: geometry collision mesh filename=file:///home/ziye01/rfmove/resources/tobor/tobor_descriptio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 scale=0.001 0.001 0.001; visual mesh filename=file:///home/ziye01/rfmove/resources/tobor/tobor_descriptio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 scale=.001 0.001 0.001
- link left_arm_link5: geometry collision mesh filename=file:///home/ziye01/rfmove/resources/tobor/tobor_descriptio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 scale=0.001 0.001 0.001; visual mesh filename=file:///home/ziye01/rfmove/resources/tobor/tobor_descriptio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 scale=0.001 0.001 0.001
- link left_arm_link6: geometry collision mesh filename=file:///home/ziye01/rfmove/resources/tobor/tobor_descriptio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 scale=0.001 0.001 0.001; visual mesh filename=file:///home/ziye01/rfmove/resources/tobor/tobor_descriptio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 scale=0.001 0.001 0.001
- link left_arm_link7: geometry collision mesh filename=file:///home/ziye01/rfmove/resources/tobor/tobor_descriptio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 scale=0.001 0.001 0.001; visual mesh filename=file:///home/ziye01/rfmove/resources/tobor/tobor_descriptio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 scale=0.001 0.001 0.001
- link left_inner_finger_left: geometry collision mesh filename=file:///home/ziye01/rfmove/resources/tobor/tobor_descriptio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 scale=0.001 0.001 0.001; visual mesh filename=file:///home/ziye01/rfmove/resources/tobor/tobor_descriptio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 scale=0.001 0.001 0.001
- link left_inner_finger_right: geometry collision mesh filename=file:///home/ziye01/rfmove/resources/tobor/tobor_descriptio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 scale=0.001 0.001 0.001; visual mesh filename=file:///home/ziye01/rfmove/resources/tobor/tobor_descriptio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 scale=0.001 0.001 0.001
- link left_inner_knuckle_left: geometry collision mesh filename=file:///home/ziye01/rfmove/resources/tobor/tobor_descriptio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 scale=0.001 0.001 0.001; visual mesh filename=file:///home/ziye01/rfmove/resources/tobor/tobor_descriptio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 scale=0.001 0.001 0.001
- link left_inner_knuckle_right: geometry collision mesh filename=file:///home/ziye01/rfmove/resources/tobor/tobor_descriptio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 scale=0.001 0.001 0.001; visual mesh filename=file:///home/ziye01/rfmove/resources/tobor/tobor_descriptio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 scale=0.001 0.001 0.001
- link left_outer_finger_left: geometry collision mesh filename=file:///home/ziye01/rfmove/resources/tobor/tobor_descriptio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 scale=0.001 0.001 0.001; visual mesh filename=file:///home/ziye01/rfmove/resources/tobor/tobor_descriptio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 scale=0.001 0.001 0.001
- link left_outer_finger_right: geometry collision mesh filename=file:///home/ziye01/rfmove/resources/tobor/tobor_descriptio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 scale=0.001 0.001 0.001; visual mesh filename=file:///home/ziye01/rfmove/resources/tobor/tobor_descriptio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 scale=0.001 0.001 0.001
- link left_outer_knuckle_left: geometry collision mesh filename=file:///home/ziye01/rfmove/resources/tobor/tobor_descriptio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 scale=0.001 0.001 0.001; visual mesh filename=file:///home/ziye01/rfmove/resources/tobor/tobor_descriptio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 scale=0.001 0.001 0.001
- link left_outer_knuckle_right: mass None -> 0.00853198276973456; geometry collision mesh filename=file:///home/ziye01/rfmove/resources/tobor/tobor_descriptio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 scale=0.001 0.001 0.001; visual mesh filename=file:///home/ziye01/rfmove/resources/tobor/tobor_descriptio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 scale=0.001 0.001 0.001
- link left_wheel_link: geometry collision mesh filename=file:///home/ziye01/rfmove/resources/tobor/tobor_descriptio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; visual mesh filename=file:///home/ziye01/rfmove/resources/tobor/tobor_descriptio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
- link lifting_rod_link: geometry collision mesh filename=file:///home/ziye01/rfmove/resources/tobor/tobor_descriptio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; visual mesh filename=file:///home/ziye01/rfmove/resources/tobor/tobor_descriptio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
- link power_link: geometry collision mesh filename=file:///home/ziye01/rfmove/resources/tobor/tobor_descriptio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; visual mesh filename=file:///home/ziye01/rfmove/resources/tobor/tobor_descriptio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
- link rear_lower_body_link: geometry collision mesh filename=file:///home/ziye01/rfmove/resources/tobor/tobor_descriptio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; visual mesh filename=file:///home/ziye01/rfmove/resources/tobor/tobor_descriptio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
- link rear_upper_body_link: geometry collision mesh filename=file:///home/ziye01/rfmove/resources/tobor/tobor_descriptio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; visual mesh filename=file:///home/ziye01/rfmove/resources/tobor/tobor_descriptio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
- link right_arm_base: geometry collision mesh filename=file:///home/ziye01/rfmove/resources/tobor/tobor_descriptio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 scale=0.001 0.001 0.001; visual mesh filename=file:///home/ziye01/rfmove/resources/tobor/tobor_descriptio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 scale=0.001 0.001 0.001
- link right_arm_link1: geometry collision mesh filename=file:///home/ziye01/rfmove/resources/tobor/tobor_descriptio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 scale=0.001 0.001 0.001; visual mesh filename=file:///home/ziye01/rfmove/resources/tobor/tobor_descriptio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 scale=0.001 0.001 0.001
- link right_arm_link2: geometry collision mesh filename=file:///home/ziye01/rfmove/resources/tobor/tobor_descriptio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 scale=0.001 0.001 0.001; visual mesh filename=file:///home/ziye01/rfmove/resources/tobor/tobor_descriptio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 scale=0.001 0.001 0.001
- link right_arm_link3: geometry collision mesh filename=file:///home/ziye01/rfmove/resources/tobor/tobor_descriptio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 scale=0.001 0.001 0.001; visual mesh filename=file:///home/ziye01/rfmove/resources/tobor/tobor_descriptio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 scale=0.001 0.001 0.001
- link right_arm_link4: geometry collision mesh filename=file:///home/ziye01/rfmove/resources/tobor/tobor_descriptio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 scale=0.001 0.001 0.001; visual mesh filename=file:///home/ziye01/rfmove/resources/tobor/tobor_descriptio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 scale=.001 0.001 0.001
- link right_arm_link5: geometry collision mesh filename=file:///home/ziye01/rfmove/resources/tobor/tobor_descriptio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 scale=0.001 0.001 0.001; visual mesh filename=file:///home/ziye01/rfmove/resources/tobor/tobor_descriptio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 scale=0.001 0.001 0.001
- link right_arm_link6: geometry collision mesh filename=file:///home/ziye01/rfmove/resources/tobor/tobor_descriptio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 scale=0.001 0.001 0.001; visual mesh filename=file:///home/ziye01/rfmove/resources/tobor/tobor_descriptio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 scale=0.001 0.001 0.001
- link right_arm_link7: geometry collision mesh filename=file:///home/ziye01/rfmove/resources/tobor/tobor_descriptio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 scale=0.001 0.001 0.001; visual mesh filename=file:///home/ziye01/rfmove/resources/tobor/tobor_descriptio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 scale=0.001 0.001 0.001
- link right_inner_finger_left: geometry collision mesh filename=file:///home/ziye01/rfmove/resources/tobor/tobor_descriptio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 scale=0.001 0.001 0.001; visual mesh filename=file:///home/ziye01/rfmove/resources/tobor/tobor_descriptio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 scale=0.001 0.001 0.001
- link right_inner_finger_right: geometry collision mesh filename=file:///home/ziye01/rfmove/resources/tobor/tobor_descriptio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 scale=0.001 0.001 0.001; visual mesh filename=file:///home/ziye01/rfmove/resources/tobor/tobor_descriptio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 scale=0.001 0.001 0.001
- link right_inner_knuckle_left: geometry collision mesh filename=file:///home/ziye01/rfmove/resources/tobor/tobor_descriptio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 scale=0.001 0.001 0.001; visual mesh filename=file:///home/ziye01/rfmove/resources/tobor/tobor_descriptio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 scale=0.001 0.001 0.001
- link right_inner_knuckle_right: geometry collision mesh filename=file:///home/ziye01/rfmove/resources/tobor/tobor_descriptio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 scale=0.001 0.001 0.001; visual mesh filename=file:///home/ziye01/rfmove/resources/tobor/tobor_descriptio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 scale=0.001 0.001 0.001
- link right_outer_finger_left: geometry collision mesh filename=file:///home/ziye01/rfmove/resources/tobor/tobor_descriptio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 scale=0.001 0.001 0.001; visual mesh filename=file:///home/ziye01/rfmove/resources/tobor/tobor_descriptio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 scale=0.001 0.001 0.001
- link right_outer_finger_right: geometry collision mesh filename=file:///home/ziye01/rfmove/resources/tobor/tobor_descriptio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 scale=0.001 0.001 0.001; visual mesh filename=file:///home/ziye01/rfmove/resources/tobor/tobor_descriptio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 scale=0.001 0.001 0.001
- link right_outer_knuckle_left: geometry collision mesh filename=file:///home/ziye01/rfmove/resources/tobor/tobor_descriptio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 scale=0.001 0.001 0.001; visual mesh filename=file:///home/ziye01/rfmove/resources/tobor/tobor_descriptio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 scale=0.001 0.001 0.001
- link right_outer_knuckle_right: geometry collision mesh filename=file:///home/ziye01/rfmove/resources/tobor/tobor_descriptio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 scale=0.001 0.001 0.001; visual mesh filename=file:///home/ziye01/rfmove/resources/tobor/tobor_descriptio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 scale=0.001 0.001 0.001
- link right_wheel_link: geometry collision mesh filename=file:///home/ziye01/rfmove/resources/tobor/tobor_descriptio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; visual mesh filename=file:///home/ziye01/rfmove/resources/tobor/tobor_descriptio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
- link robotiq_arg2f_base_link_left: geometry collision mesh filename=file:///home/ziye01/rfmove/resources/tobor/tobor_descriptio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; visual mesh filename=file:///home/ziye01/rfmove/resources/tobor/tobor_descriptio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 scale=0.001 0.001 0.001
- link robotiq_arg2f_base_link_right: geometry collision mesh filename=file:///home/ziye01/rfmove/resources/tobor/tobor_descriptio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; visual mesh filename=file:///home/ziye01/rfmove/resources/tobor/tobor_descriptio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 scale=0.001 0.001 0.001
- link sound_link: geometry collision mesh filename=file:///home/ziye01/rfmove/resources/tobor/tobor_descriptio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; visual mesh filename=file:///home/ziye01/rfmove/resources/tobor/tobor_descriptio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
- link support_plate_link: geometry collision mesh filename=file:///home/ziye01/rfmove/resources/tobor/tobor_descriptio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; visual mesh filename=file:///home/ziye01/rfmove/resources/tobor/tobor_descriptio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
- link turn_to_link: geometry collision mesh filename=file:///home/ziye01/rfmove/resources/tobor/tobor_descriptio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; visual mesh filename=file:///home/ziye01/rfmove/resources/tobor/tobor_descriptio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
Joints:
- joint tobor_grasptarget_hand_left: origin xyz=0 0 0.05 rpy=0 0 0 -> xyz=0 0 0.04 rpy=0 0 0
- joint tobor_grasptarget_hand_right: origin xyz=0 0 0.05 rpy=0 0 0 -> xyz=0 0 0.00 rpy=0 0 0
