Commit message: 6_30

File: resources/tobor/tobor_description/tobor.urdf (robot description, URDF)
Before this commit: robot r300, 69 links, 68 joints
Links:
- removed link robotiq_85_base_link_left
- removed link robotiq_85_base_link_right
- removed link robotiq_85_coupling_left
- removed link robotiq_85_coupling_right
- removed link robotiq_85_left_finger_link_left
- removed link robotiq_85_left_finger_link_right
- removed link robotiq_85_left_finger_tip_link_left
- removed link robotiq_85_left_finger_tip_link_right
- removed link robotiq_85_left_inner_knuckle_link_left
- removed link robotiq_85_left_inner_knuckle_link_right
- removed link robotiq_85_left_knuckle_link_left
- removed link robotiq_85_left_knuckle_link_right
- removed link robotiq_85_right_finger_link_left
- removed link robotiq_85_right_finger_link_right
- removed link robotiq_85_right_finger_tip_link_left
- removed link robotiq_85_right_finger_tip_link_right
- removed link robotiq_85_right_inner_knuckle_link_left
- removed link robotiq_85_right_inner_knuckle_link_right
- removed link robotiq_85_right_knuckle_link_left
- removed link robotiq_85_right_knuckle_link_right
- added link left_inner_finger_left; collision mesh filename=file:///home/ziye01/rfmove/resources/tobor/tobor_descriptio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 scale=0.001 0.001 0.001; visual mesh filename=file:///home/ziye01/rfmove/resources/tobor/tobor_descriptio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 scale=0.001 0.001 0.001
- added link left_inner_finger_pad_left; collision box size=0.022 0.00635 0.0375; visual box size=0.022 0.00635 0.0375
- added link left_inner_finger_pad_right; collision box size=0.022 0.00635 0.0375; visual box size=0.022 0.00635 0.0375
- added link left_inner_finger_right; collision mesh filename=file:///home/ziye01/rfmove/resources/tobor/tobor_descriptio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 scale=0.001 0.001 0.001; visual mesh filename=file:///home/ziye01/rfmove/resources/tobor/tobor_descriptio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 scale=0.001 0.001 0.001
- added link left_inner_knuckle_left; collision mesh filename=file:///home/ziye01/rfmove/resources/tobor/tobor_descriptio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 scale=0.001 0.001 0.001; visual mesh filename=file:///home/ziye01/rfmove/resources/tobor/tobor_descriptio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 scale=0.001 0.001 0.001
- added link left_inner_knuckle_right; collision mesh filename=file:///home/ziye01/rfmove/resources/tobor/tobor_descriptio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 scale=0.001 0.001 0.001; visual mesh filename=file:///home/ziye01/rfmove/resources/tobor/tobor_descriptio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 scale=0.001 0.001 0.001
- added link left_outer_finger_left; collision mesh filename=file:///home/ziye01/rfmove/resources/tobor/tobor_descriptio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 scale=0.001 0.001 0.001; visual mesh filename=file:///home/ziye01/rfmove/resources/tobor/tobor_descriptio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 scale=0.001 0.001 0.001
- added link left_outer_finger_right; collision mesh filename=file:///home/ziye01/rfmove/resources/tobor/tobor_descriptio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 scale=0.001 0.001 0.001; visual mesh filename=file:///home/ziye01/rfmove/resources/tobor/tobor_descriptio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 scale=0.001 0.001 0.001
- added link left_outer_knuckle_left; collision mesh filename=file:///home/ziye01/rfmove/resources/tobor/tobor_descriptio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 scale=0.001 0.001 0.001; visual mesh filename=file:///home/ziye01/rfmove/resources/tobor/tobor_descriptio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 scale=0.001 0.001 0.001
- added link left_outer_knuckle_right; collision mesh filename=file:///home/ziye01/rfmove/resources/tobor/tobor_descriptio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 scale=0.001 0.001 0.001; visual mesh filename=file:///home/ziye01/rfmove/resources/tobor/tobor_descriptio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 scale=0.001 0.001 0.001
- added link right_inner_finger_left; collision mesh filename=file:///home/ziye01/rfmove/resources/tobor/tobor_descriptio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 scale=0.001 0.001 0.001; visual mesh filename=file:///home/ziye01/rfmove/resources/tobor/tobor_descriptio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 scale=0.001 0.001 0.001
- added link right_inner_finger_pad_left; collision box size=0.022 0.00635 0.0375; visual box size=0.022 0.00635 0.0375
- added link right_inner_finger_pad_right; collision box size=0.022 0.00635 0.0375; visual box size=0.022 0.00635 0.0375
- added link right_inner_finger_right; collision mesh filename=file:///home/ziye01/rfmove/resources/tobor/tobor_descriptio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 scale=0.001 0.001 0.001; visual mesh filename=file:///home/ziye01/rfmove/resources/tobor/tobor_descriptio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 scale=0.001 0.001 0.001
- added link right_inner_knuckle_left; collision mesh filename=file:///home/ziye01/rfmove/resources/tobor/tobor_descriptio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 scale=0.001 0.001 0.001; visual mesh filename=file:///home/ziye01/rfmove/resources/tobor/tobor_descriptio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 scale=0.001 0.001 0.001
- added link right_inner_knuckle_right; collision mesh filename=file:///home/ziye01/rfmove/resources/tobor/tobor_descriptio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 scale=0.001 0.001 0.001; visual mesh filename=file:///home/ziye01/rfmove/resources/tobor/tobor_descriptio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 scale=0.001 0.001 0.001
- added link right_outer_finger_left; collision mesh filename=file:///home/ziye01/rfmove/resources/tobor/tobor_descriptio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 scale=0.001 0.001 0.001; visual mesh filename=file:///home/ziye01/rfmove/resources/tobor/tobor_descriptio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 scale=0.001 0.001 0.001
- added link right_outer_finger_right; collision mesh filename=file:///home/ziye01/rfmove/resources/tobor/tobor_descriptio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 scale=0.001 0.001 0.001; visual mesh filename=file:///home/ziye01/rfmove/resources/tobor/tobor_descriptio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 scale=0.001 0.001 0.001
- added link right_outer_knuckle_left; collision mesh filename=file:///home/ziye01/rfmove/resources/tobor/tobor_descriptio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 scale=0.001 0.001 0.001; visual mesh filename=file:///home/ziye01/rfmove/resources/tobor/tobor_descriptio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 scale=0.001 0.001 0.001
- added link right_outer_knuckle_right; collision mesh filename=file:///home/ziye01/rfmove/resources/tobor/tobor_descriptio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 scale=0.001 0.001 0.001; visual mesh filename=file:///home/ziye01/rfmove/resources/tobor/tobor_descriptio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 scale=0.001 0.001 0.001
- added link robotiq_arg2f_base_link_left, mass 0.22652; collision mesh filename=file:///home/ziye01/rfmove/resources/tobor/tobor_descriptio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; visual mesh filename=file:///home/ziye01/rfmove/resources/tobor/tobor_descriptio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 scale=0.001 0.001 0.001
- added link robotiq_arg2f_base_link_right, mass 0.22652; collision mesh filename=file:///home/ziye01/rfmove/resources/tobor/tobor_descriptio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; visual mesh filename=file:///home/ziye01/rfmove/resources/tobor/tobor_descriptio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 scale=0.001 0.001 0.001
Joints:
- removed joint robotiq_85_base_joint_left
- removed joint robotiq_85_base_joint_right
- removed joint robotiq_85_left_finger_joint_left
- removed joint robotiq_85_left_finger_joint_right
- removed joint robotiq_85_left_finger_tip_joint_left
- removed joint robotiq_85_left_finger_tip_joint_right
- removed joint robotiq_85_left_inner_knuckle_joint_left
- removed joint robotiq_85_left_inner_knuckle_joint_right
- removed joint robotiq_85_left_knuckle_joint_left
- removed joint robotiq_85_left_knuckle_joint_right
- removed joint robotiq_85_right_finger_joint_left
- removed joint robotiq_85_right_finger_joint_right
- removed joint robotiq_85_right_finger_tip_joint_left
- removed joint robotiq_85_right_finger_tip_joint_right
- removed joint robotiq_85_right_inner_knuckle_joint_left
- removed joint robotiq_85_right_inner_knuckle_joint_right
- removed joint robotiq_85_right_knuckle_joint_left
- removed joint robotiq_85_right_knuckle_joint_right
- added joint finger_joint_left: type revolute, parent robotiq_arg2f_base_link_left, child left_outer_knuckle_left, origin xyz=0 -0.0306011 0.054904 rpy=0 0 3.141592653589793, axis 1 0 0, limit lower=0 upper=0.8 effort=1000 velocity=2.0
- added joint finger_joint_right: type revolute, parent robotiq_arg2f_base_link_right, child left_outer_knuckle_right, origin xyz=0 -0.0306011 0.054904 rpy=0 0 3.141592653589793, axis 1 0 0, limit lower=0 upper=0.8 effort=1000 velocity=2.0
- added joint left_inner_finger_joint_left: type revolute, parent left_outer_finger_left, child left_inner_finger_left, origin xyz=0 0.0061 0.0471 rpy=0 0 0, axis 1 0 0, limit lower=0 upper=0.8757 effort=1000 velocity=2.0, mimic joint=finger_joint_left multiplier=-1 offset=0
- added joint left_inner_finger_joint_right: type revolute, parent left_outer_finger_right, child left_inner_finger_right, origin xyz=0 0.0061 0.0471 rpy=0 0 0, axis 1 0 0, limit lower=0 upper=0.8757 effort=1000 velocity=2.0, mimic joint=finger_joint_right multiplier=-1 offset=0
- added joint left_inner_finger_pad_joint_left: type fixed, parent left_inner_finger_left, child left_inner_finger_pad_left, origin xyz=0 -0.0220203446692936 0.03242 rpy=0 0 0, axis 0 0 1
- added joint left_inner_finger_pad_joint_right: type fixed, parent left_inner_finger_right, child left_inner_finger_pad_right, origin xyz=0 -0.0220203446692936 0.03242 rpy=0 0 0, axis 0 0 1
- added joint left_inner_knuckle_joint_left: type revolute, parent robotiq_arg2f_base_link_left, child left_inner_knuckle_left, origin xyz=0 -0.0127 0.06142 rpy=0 0 3.141592653589793, axis 1 0 0, limit lower=0 upper=0.8757 effort=1000 velocity=2.0, mimic joint=finger_joint_left multiplier=1 offset=0
- added joint left_inner_knuckle_joint_right: type revolute, parent robotiq_arg2f_base_link_right, child left_inner_knuckle_right, origin xyz=0 -0.0127 0.06142 rpy=0 0 3.141592653589793, axis 1 0 0, limit lower=0 upper=0.8757 effort=1000 velocity=2.0, mimic joint=finger_joint_right multiplier=1 offset=0
- added joint left_outer_finger_joint_left: type fixed, parent left_outer_knuckle_left, child left_outer_finger_left, origin xyz=0 0.0315 -0.0041 rpy=0 0 0, axis 1 0 0
- added joint left_outer_finger_joint_right: type fixed, parent left_outer_knuckle_right, child left_outer_finger_right, origin xyz=0 0.0315 -0.0041 rpy=0 0 0, axis 1 0 0
- added joint right_inner_finger_joint_left: type revolute, parent right_outer_finger_left, child right_inner_finger_left, origin xyz=0 0.0061 0.0471 rpy=0 0 0, axis 1 0 0, limit lower=0 upper=0.8757 effort=1000 velocity=2.0, mimic joint=finger_joint_left multiplier=-1 offset=0
- added joint right_inner_finger_joint_right: type revolute, parent right_outer_finger_right, child right_inner_finger_right, origin xyz=0 0.0061 0.0471 rpy=0 0 0, axis 1 0 0, limit lower=0 upper=0.8757 effort=1000 velocity=2.0, mimic joint=finger_joint_right multiplier=-1 offset=0
- added joint right_inner_finger_pad_joint_left: type fixed, parent right_inner_finger_left, child right_inner_finger_pad_left, origin xyz=0 -0.0220203446692936 0.03242 rpy=0 0 0, axis 0 0 1
- added joint right_inner_finger_pad_joint_right: type fixed, parent right_inner_finger_right, child right_inner_finger_pad_right, origin xyz=0 -0.0220203446692936 0.03242 rpy=0 0 0, axis 0 0 1
- added joint right_inner_knuckle_joint_left: type revolute, parent robotiq_arg2f_base_link_left, child right_inner_knuckle_left, origin xyz=0 0.0127 0.06142 rpy=0 0 0.0, axis 1 0 0, limit lower=0 upper=0.8757 effort=1000 velocity=2.0, mimic joint=finger_joint_left multiplier=1 offset=0
- added joint right_inner_knuckle_joint_right: type revolute, parent robotiq_arg2f_base_link_right, child right_inner_knuckle_right, origin xyz=0 0.0127 0.06142 rpy=0 0 0.0, axis 1 0 0, limit lower=0 upper=0.8757 effort=1000 velocity=2.0, mimic joint=finger_joint_right multiplier=1 offset=0
- added joint right_outer_finger_joint_left: type fixed, parent right_outer_knuckle_left, child right_outer_finger_left, origin xyz=0 0.0315 -0.0041 rpy=0 0 0, axis 1 0 0
- added joint right_outer_finger_joint_right: type fixed, parent right_outer_knuckle_right, child right_outer_finger_right, origin xyz=0 0.0315 -0.0041 rpy=0 0 0, axis 1 0 0
- added joint right_outer_knuckle_joint_left: type revolute, parent robotiq_arg2f_base_link_left, child right_outer_knuckle_left, origin xyz=0 0.0306011 0.054904 rpy=0 0 0, axis 1 0 0, limit lower=0 upper=0.81 effort=1000 velocity=2.0, mimic joint=finger_joint_left multiplier=1 offset=0
- added joint right_outer_knuckle_joint_right: type revolute, parent robotiq_arg2f_base_link_right, child right_outer_knuckle_right, origin xyz=0 0.0306011 0.054904 rpy=0 0 0, axis 1 0 0, limit lower=0 upper=0.81 effort=1000 velocity=2.0, mimic joint=finger_joint_right multiplier=1 offset=0
- joint tobor_grasptarget_hand_left: child robotiq_85_coupling_left -> robotiq_arg2f_base_link_left
- joint tobor_grasptarget_hand_right: child robotiq_85_coupling_right -> robotiq_arg2f_base_link_right

Commit message: 6_30

File: resources/tobor/tobor_description/tobor.urdf (robot description, URDF)
Before this commit: robot r300, 71 links, 70 joints
Links:
- link base_link: mass None -> 0.0001
Joints:
- joint tobor_grasptarget_hand_left: origin xyz=0 0 0.0 rpy=0 0 0 -> xyz=0 0 0.05 rpy=0 0 0
- joint tobor_grasptarget_hand_right: origin xyz=0 0 0.0 rpy=0 0 0 -> xyz=0 0 0.05 rpy=0 0 0
