Commit message: rfmove_7_4_1

File: resources/tobor_arm/tobor_arm_description/urdf/tobor_arm.urdf (robot description, URDF)
Before this commit: robot r300, 8 links, 7 joints
Links:
- link left_arm_base: geometry collision mesh filename=file:///home/ziye01/rfmove/resources/tobor_arm/tobor_descri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 scale=0.001 0.001 0.001; visual mesh filename=file:///home/ziye01/rfmove/resources/tobor_arm/tobor_descri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 scale=0.001 0.001 0.001
- link left_arm_link1: geometry collision mesh filename=file:///home/ziye01/rfmove/resources/tobor_arm/tobor_descri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 scale=0.001 0.001 0.001; visual mesh filename=file:///home/ziye01/rfmove/resources/tobor_arm/tobor_descri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 scale=0.001 0.001 0.001
- link left_arm_link2: geometry collision mesh filename=file:///home/ziye01/rfmove/resources/tobor_arm/tobor_descri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 scale=0.001 0.001 0.001; visual mesh filename=file:///home/ziye01/rfmove/resources/tobor_arm/tobor_descri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 scale=0.001 0.001 0.001
- link left_arm_link3: geometry collision mesh filename=file:///home/ziye01/rfmove/resources/tobor_arm/tobor_descri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 scale=0.001 0.001 0.001; visual mesh filename=file:///home/ziye01/rfmove/resources/tobor_arm/tobor_descri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 scale=0.001 0.001 0.001
- link left_arm_link4: geometry collision mesh filename=file:///home/ziye01/rfmove/resources/tobor_arm/tobor_descri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 scale=0.001 0.001 0.001; visual mesh filename=file:///home/ziye01/rfmove/resources/tobor_arm/tobor_descri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 scale=.001 0.001 0.001
- link left_arm_link5: geometry collision mesh filename=file:///home/ziye01/rfmove/resources/tobor_arm/tobor_descri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 scale=0.001 0.001 0.001; visual mesh filename=file:///home/ziye01/rfmove/resources/tobor_arm/tobor_descri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 scale=0.001 0.001 0.001
- link left_arm_link6: geometry collision mesh filename=file:///home/ziye01/rfmove/resources/tobor_arm/tobor_descri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 scale=0.001 0.001 0.001; visual mesh filename=file:///home/ziye01/rfmove/resources/tobor_arm/tobor_descri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 scale=0.001 0.001 0.001
- link left_arm_link7: geometry collision mesh filename=file:///home/ziye01/rfmove/resources/tobor_arm/tobor_descri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 scale=0.001 0.001 0.001; visual mesh filename=file:///home/ziye01/rfmove/resources/tobor_arm/tobor_descri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 scale=0.001 0.001 0.001

Commit message: rfmove-7-4

File: resources/tobor_arm/tobor_arm_description/urdf/tobor_arm.urdf (robot description, URDF)
Before this commit: robot r300, 8 links, 7 joints
Links:
- link left_arm_base: geometry collision mesh filename=file:///home/lees/linux_bak/rfmove/resources/tobor_arm/tobo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 scale=0.001 0.001 0.001; visual mesh filename=file:///home/lees/linux_bak/rfmove/resources/tobor_arm/tobo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 scale=0.001 0.001 0.001
- link left_arm_link1: geometry collision mesh filename=file:///home/lees/linux_bak/rfmove/resources/tobor_arm/tobo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 scale=0.001 0.001 0.001; visual mesh filename=file:///home/lees/linux_bak/rfmove/resources/tobor_arm/tobo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 scale=0.001 0.001 0.001
- link left_arm_link2: geometry collision mesh filename=file:///home/lees/linux_bak/rfmove/resources/tobor_arm/tobo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 scale=0.001 0.001 0.001; visual mesh filename=file:///home/lees/linux_bak/rfmove/resources/tobor_arm/tobo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 scale=0.001 0.001 0.001
- link left_arm_link3: geometry collision mesh filename=file:///home/lees/linux_bak/rfmove/resources/tobor_arm/tobo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 scale=0.001 0.001 0.001; visual mesh filename=file:///home/lees/linux_bak/rfmove/resources/tobor_arm/tobo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 scale=0.001 0.001 0.001
- link left_arm_link4: geometry collision mesh filename=file:///home/lees/linux_bak/rfmove/resources/tobor_arm/tobo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 scale=0.001 0.001 0.001; visual mesh filename=file:///home/lees/linux_bak/rfmove/resources/tobor_arm/tobo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 scale=.001 0.001 0.001
- link left_arm_link5: geometry collision mesh filename=file:///home/lees/linux_bak/rfmove/resources/tobor_arm/tobo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 scale=0.001 0.001 0.001; visual mesh filename=file:///home/lees/linux_bak/rfmove/resources/tobor_arm/tobo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 scale=0.001 0.001 0.001
- link left_arm_link6: geometry collision mesh filename=file:///home/lees/linux_bak/rfmove/resources/tobor_arm/tobo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 scale=0.001 0.001 0.001; visual mesh filename=file:///home/lees/linux_bak/rfmove/resources/tobor_arm/tobo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 scale=0.001 0.001 0.001
- link left_arm_link7: geometry collision mesh filename=file:///home/lees/linux_bak/rfmove/resources/tobor_arm/tobo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 scale=0.001 0.001 0.001; visual mesh filename=file:///home/lees/linux_bak/rfmove/resources/tobor_arm/tobo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 scale=0.001 0.001 0.001

Commit message: rfmove_7_4_2

File: resources/tobor_arm/tobor_arm_description/urdf/tobor_arm.urdf (robot description, URDF)
Before this commit: robot r300, 8 links, 7 joints
Links:
- link left_arm_base: geometry collision mesh filename=package://tobor_arm_description/meshes/xmate3/meshes/collis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 scale=0.001 0.001 0.001; visual mesh filename=package://tobor_arm_description/meshes/xmate3/meshes/visual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 scale=0.001 0.001 0.001
- link left_arm_link1: geometry collision mesh filename=package://tobor_arm_description/meshes/xmate3/meshes/collis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 scale=0.001 0.001 0.001; visual mesh filename=package://tobor_arm_description/meshes/xmate3/meshes/visual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 scale=0.001 0.001 0.001
- link left_arm_link2: geometry collision mesh filename=package://tobor_arm_description/meshes/xmate3/meshes/collis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 scale=0.001 0.001 0.001; visual mesh filename=package://tobor_arm_description/meshes/xmate3/meshes/visual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 scale=0.001 0.001 0.001
- link left_arm_link3: geometry collision mesh filename=package://tobor_arm_description/meshes/xmate3/meshes/collis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 scale=0.001 0.001 0.001; visual mesh filename=package://tobor_arm_description/meshes/xmate3/meshes/visual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 scale=0.001 0.001 0.001
- link left_arm_link4: geometry collision mesh filename=package://tobor_arm_description/meshes/xmate3/meshes/collis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 scale=0.001 0.001 0.001; visual mesh filename=package://tobor_arm_description/meshes/xmate3/meshes/visual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 scale=.001 0.001 0.001
- link left_arm_link5: geometry collision mesh filename=package://tobor_arm_description/meshes/xmate3/meshes/collis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 scale=0.001 0.001 0.001; visual mesh filename=package://tobor_arm_description/meshes/xmate3/meshes/visual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 scale=0.001 0.001 0.001
- link left_arm_link6: geometry collision mesh filename=package://tobor_arm_description/meshes/xmate3/meshes/collis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 scale=0.001 0.001 0.001; visual mesh filename=package://tobor_arm_description/meshes/xmate3/meshes/visual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 scale=0.001 0.001 0.001
- link left_arm_link7: geometry collision mesh filename=package://tobor_arm_description/meshes/xmate3/meshes/collis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 scale=0.001 0.001 0.001; visual mesh filename=package://tobor_arm_description/meshes/xmate3/meshes/visual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 scale=0.001 0.001 0.001
